File: EV_Charger_KiCad_Prototype/EV_Charger_KiCad_Prototype.kicad_pcb (KiCad board)
At the start: 2 copper layers, 0 parts

Commit message: Simplify main KiCad project files for standard opening
Other:
- board outline added: 110 x 70 mm
Changed lines of the file:
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@@
-(kicad_pcb (version 20240108) (generator "pcbnew")
+(kicad_pcb (version 20221018) (generator pcbnew)
   (general
     (thickness 1.6)
@@
     (nets 0)
   )
-  (page A4)
+  (paper "A4")
   (layers
     (0 F.Cu signal)
@@
   (setup
     (pad_to_mask_clearance 0.05)
-    (pcbplotparams
-      (layerselection 0x010fc_ffffffff)
-      (plot_on_all_layers_selection 0x0000000)
-      (disableapertmacros false)
-      (usegerberextensions false)
-      (usegerberattributes true)
-      (usegerberadvancedattributes true)
-      (creategerberjobfile false)
-      (dashed_line_dash_ratio 12.000000)
-      (dashed_line_gap_ratio 3.000000)
-      (svgprecision 6)
-    )
   )
+  (gr_rect (start 10 10) (end 120 80) (layer "Edge.Cuts") (width 0.1))
 )
